File: diode555/diode555.kicad_sch (KiCad schematic)
At the start: 0 parts

Commit message: schematic
Parts:
- added C1: 10u, Capacitor_THT:C_Disc_D5.0mm_W2.5mm_P5.00mm, symbol Device:C
- added C2: 10n, Capacitor_THT:C_Disc_D5.0mm_W2.5mm_P5.00mm, symbol Device:C
- added D1: LED, LED_THT:LED_D5.0mm, symbol Device:LED
- added R1, R3: 1k, Resistor_THT:R_Axial_DIN0207_L6.3mm_D2.5mm_P10.16mm_Horizontal, symbol Device:R
- added R2: 100k, Resistor_THT:R_Axial_DIN0207_L6.3mm_D2.5mm_P10.16mm_Horizontal, symbol Device:R
- added U1: NE555P, Package_DIP:DIP-8_W7.62mm, symbol Timer:NE555P
Connections:
- new net: R1.2, R2.1, U1.7 (DISCH)
- new net: C1.1, R2.2, U1.2 (TRIG), U1.6 (THRES)
- new net: C2.1, U1.5 (CONT)
- new net: D1.2 (A), R3.2
- new net: R3.1, U1.3 (OUT)
- new net +5V: R1.1, U1.4 (~{RST}), U1.8 (VCC)
- new net GND: C1.2, C2.2, D1.1 (K), U1.1 (GND)

Commit message: pcb intro
Parts:
- added J1: PWR Connector, Connector_PinHeader_2.54mm:PinHeader_2x01_P2.54mm_Vertical, symbol Connector_Generic:Conn_02x01
Connections:
- net +5V: now also J1.1 (Pin_1)
- net GND: now also J1.2 (Pin_2)
Other:
- company: (none) -> Marcel Siwiela
- title: (none) -> NE555 with LED
- moved on the sheet: C1, C2, D1, R1, R2, R3, U1
