File: diode555/diode555.kicad_pcb (KiCad board)
At the start: 4 copper layers, 40 x 22 mm, 8 parts, among them J1 PWR Connector, U1 NE555P

Commit message: some routes
Routing:
- net +5V: track 0.00 -> 36.9 mm
- net Net-(D1-A): track 0.00 -> 12.7 mm
- net Net-(U1-THRES): track 0.00 -> 10.7 mm
- net Net-(U1-OUT): track 0.00 -> 10.6 mm
- net Net-(U1-CONT): track 0.00 -> 5.77 mm
- net Net-(U1-DISCH): track 0.00 -> 5.21 mm
Changed lines of the file:
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@@
 		(layer "Edge.Cuts")
+	)
+	(segment
+		(start 149.92 103.58)
+		(end 152.5 101)
+		(width 0.2)
+		(layer "F.Cu")
+		(net "Net-(U1-THRES)")
+	)
+	(segment
+		(start 147.5 103.58)
+		(end 149.92 103.58)
+		(width 0.2)
+		(layer "F.Cu")
+		(net "Net-(U1-THRES)")
+	)
+	(segment
+		(start 152.5 101)
+		(end 153.945 101)
+		(width 0.2)
+		(layer "F.Cu")
+		(net "Net-(U1-THRES)")
+	)
+	(segment
+		(start 153.945 101)
+		(end 156.215 98.73)
+		(width 0.2)
+		(layer "F.Cu")
+		(net "Net-(U1-THRES)")
+	)
+	(segment
+		(start 163.835 103.81)
+		(end 166.29 103.81)
+		(width 0.2)
+		(layer "F.Cu")
+		(net "Net-(U1-CONT)")
+	)
+	(segment
+		(start 166.29 103.81)
+		(end 167.5 102.6)
+		(width 0.2)
+		(layer "F.Cu")
+		(net "Net-(U1-CONT)")
+	)
+	(segment
+		(start 167.5 102.6)
+		(end 167.5 101)
+		(width 0.2)
+		(layer "F.Cu")
+		(net "Net-(U1-CONT)")
+	)
+	(segment
+		(start 165.08 109)
+		(end 173.99 100.09)
+		(width 0.2)
+		(layer "F.Cu")
+		(net "Net-(D1-A)")
+	)
+	(segment
+		(start 173.99 100.09)
+		(end 173.99 100)
+		(width 0.2)
+		(layer "F.Cu")
+		(net "Net-(D1-A)")
+	)
+	(segment
+		(start 161.5 91)
+		(end 161.5 93.855)
+		(width 0.2)
+		(layer "F.Cu")
+		(net "+5V")
+	)
+	(segment
+		(start 163.835 96.19)
+		(end 162.41 96.19)
+		(width 0.2)
+		(layer "F.Cu")
+		(net "+5V")
+	)
+	(segment
+		(start 153.69 103.81)
+		(end 155 103.81)
+		(width 0.2)
+		(layer "F.Cu")
+		(net "+5V")
+	)
+	(segment
+		(start 162.41 96.19)
+		(end 158.6 100)
+		(width 0.2)
+		(layer "F.Cu")
+		(net "+5V")
+	)
+	(segment
+		(start 150.2 107.3)
+		(end 153.69 103.81)
+		(width 0.2)
+		(layer "F.Cu")
+		(net "+5V")
+	)
+	(segment
+		(start 158.6 100)
+		(end 155.6 100)
+		(width 0.2)
+		(layer "F.Cu")
+		(net "+5V")
+	)
+	(segment
+		(start 155 103.81)
+		(end 156.215 103.81)
+		(width 0.2)
+		(layer "F.Cu")
+		(net "+5V")
+	)
+	(segment
+		(start 145.72 107.3)
+		(end 150.2 107.3)
+		(width 0.2)
+		(layer "F.Cu")
+		(net "+5V")
+	)
+	(segment
+		(start 154.6 103.41)
+		(end 155 103.81)
+		(width 0.2)
+		(layer "F.Cu")
+		(net "+5V")
+	)
+	(segment
+		(start 142.5 104.08)
+		(end 145.72 107.3)
+		(width 0.2)
+		(layer "F.Cu")
+		(net "+5V")
+	)
+	(segment
+		(start 155.6 100)
+		(end 154.6 101)
+		(width 0.2)
+		(layer "F.Cu")
+		(net "+5V")
+	)
+	(segment
+		(start 161.5 93.855)
+		(end 163.835 96.19)
+		(width 0.2)
+		(layer "F.Cu")
+		(net "+5V")
+	)
+	(segment
+		(start 154.6 101)
+		(end 154.6 103.41)
+		(width 0.2)
+		(layer "F.Cu")
+		(net "+5V")
+	)
+	(segment
+		(start 147 93.92)
+		(end 147.5 93.42)
+		(width 0.2)
+		(layer "F.Cu")
+		(net "Net-(U1-DISCH)")
+	)
+	(segment
+		(start 142.5 93.92)
+		(end 147 93.92)
+		(width 0.2)
+		(layer "F.Cu")
+		(net "Net-(U1-DISCH)")
+	)
+	(segment
+		(start 158.3 105.62)
+		(end 158.3 102.3)
+		(width 0.2)
+		(layer "F.Cu")
+		(net "Net-(U1-OUT)")
+	)
+	(segment
+		(start 154.92 109)
+		(end 158.3 105.62)
+		(width 0.2)
+		(layer "F.Cu")
+		(net "Net-(U1-OUT)")
+	)
+	(segment
+		(start 156.545 101.6)
+		(end 156.215 101.27)
+		(width 0.2)
+		(layer "F.Cu")
+		(net "Net-(U1-OUT)")
+	)
+	(segment
+		(start 157.6 101.6)
+		(end 156.545 101.6)
+		(width 0.2)
+		(layer "F.Cu")
+		(net "Net-(U1-OUT)")
+	)
+	(segment
+		(start 158.3 102.3)
+		(end 157.6 101.6)
+		(width 0.2)
+		(layer "F.Cu")
+		(net "Net-(U1-OUT)")
 	)
 	(zone

Commit message: pcb done
Parts:
- moved C1 60.5 mm to (103.7, 65.2)
- moved C2 60.5 mm to (118.7, 65.2)
- moved D1 60.5 mm to (125.2, 61.7)
- moved J1 60.5 mm to (112.7, 55.2)
- moved R1 60.5 mm to (93.7, 68.3)
- moved R2 60.5 mm to (98.7, 57.6)
- moved U1 60.5 mm to (107.4, 60.4)
- moved R3 60.5 mm to (106.1, 73.2)
Routing:
- net Net-(U1-DISCH): track 5.21 -> 23.7 mm
- net Net-(U1-THRES): track 10.7 -> 20.2 mm, vias 0 -> 1
- net +5V: track 36.9 -> 32.3 mm
- net Net-(U1-OUT): track 10.6 -> 9.61 mm
Other:
- board text added: "+"
- board text added: "-"
- board text added: "Blink"
- board text added: "Hello World!"
- board text added: "MS 10.10.26"
- board text added: "via test :)"

Commit message: pcb changes
Parts:
- added G***: LOGO, LOGO, B.Cu at (111.4, 64.5)
- added Hole test: MountingHole_2.1mm, MountingHole:MountingHole_2.1mm, F.Cu at (119.7, 56.1)
Routing:
- removed copper zone on B.Cu, net GND
Other:
- board text added: "100k"
- board text added: "10n"
- board text added: "10u"
- board text added: "1k"
- board text added: "JLCJLCJLCJLC"
